Commit message: 08/08/2025

File: install/jetacker_description/share/jetacker_description/urdf/imu.urdf.xacro (robot description, xacro)
@@ -1,16 +1 @@
-<?xml version="1.0" encoding="utf-8"?>
-<robot name="imu" xmlns:xacro="http://ros.org/wiki/xacro">
-  <xacro:property name="M_PI" value="3.1415926535897931"/>
-  <link name="imu_link"/>
-  <joint
-    name="imu_joint"
-    type="fixed">
-    <origin
-      xyz="0 0 ${0.025 - 0.0295 + 0.0965/2 + 0.0678410821576746}"
-      rpy="0 0 -${M_PI/2}" />
-    <parent
-      link="base_link"/>
-    <child
-      link="imu_link"/>
-  </joint>
-</robot>
+/home/ubuntu/ros2_ws/build/jetacker_description/urdf/imu.urdf.xacro

File: install/jetacker_description/share/jetacker_description/urdf/inertial_matrix.xacro (robot description, xacro)
@@ -1,41 +1 @@
-<?xml version="1.0" encoding="utf-8"?>
-<robot name="inertial_matrix" xmlns:xacro="http://ros.org/wiki/xacro">
-  <xacro:property name="M_PI" value="3.1415926535897931" />
-  <!-- Macro for inertia matrix -->
-  <xacro:macro name="sphere_inertial" params="m r">
-    <inertial>
-      <mass value="${m}" />
-      <inertia
-        ixx="${2*m*r*r/5}"
-        ixy="0"
-        ixz="0"
-        iyy="${2*m*r*r/5}"
-        iyz="0"
-        izz="${2*m*r*r/5}" />
-    </inertial>
-  </xacro:macro>
-  <xacro:macro name="cylinder_inertial" params="m r h">
-    <inertial>
-      <mass value="${m}" />
-      <inertia
-        ixx="${m*(3*r*r+h*h)/12}"
-        ixy = "0"
-        ixz = "0"
-        iyy="${m*(3*r*r+h*h)/12}"
-        iyz = "0"
-        izz="${m*r*r/2}" />
-    </inertial>
-  </xacro:macro>
-  <xacro:macro name="box_inertial" params="m w h d">
-    <inertial>
-      <mass value="${m}" />
-      <inertia
-        ixx="${m*(h*h+d*d)/12}"
-        ixy = "0"
-        ixz = "0"
-        iyy="${m*(w*w+d*d)/12}"
-        iyz = "0"
-        izz="${m*(w*w+h*h)/12}" />
-    </inertial>
-  </xacro:macro>
-</robot>
+/home/ubuntu/ros2_ws/build/jetacker_description/urdf/inertial_matrix.xacro

File: install/jetacker_description/share/jetacker_description/urdf/jetacker.urdf.xacro (robot description, xacro)
@@ -1,387 +1 @@
-<?xml version="1.0" encoding="utf-8"?>
-<robot name="jetacker" xmlns:xacro="http://ros.org/wiki/xacro" >
-  <xacro:property name="M_PI"               value="3.1415926535897931"/>
-  <xacro:property name="base_link_mass"     value="1.6" />
-  <xacro:property name="base_link_w"        value="0.296"/>
-  <xacro:property name="base_link_h"        value="0.16"/>
-  <xacro:property name="base_link_d"        value="0.126"/>
-  <xacro:property name="body_link_mass"     value="1.6" />
-  <xacro:property name="body_link_w"        value="0.22"/>
-  <xacro:property name="body_link_h"        value="0.17"/>
-  <xacro:property name="body_link_d"        value="0.095"/>
-  <xacro:property name="wheel_link_mass"    value="8.0" />
-  <xacro:property name="wheel_link_radius"  value="0.05"/>
-  <xacro:property name="wheel_link_length"  value="0.039"/>
-  <link name="base_footprint"/>
-  <joint name="base_joint" type="fixed">
-    <parent link="base_footprint"/>
-    <child link="base_link"/>
-    <origin xyz="0.0 0.0 0" rpy="0 0 0"/>
-  </joint>
-  <link
-    name="base_link">
-    <xacro:box_inertial m="${base_link_mass}" w="${base_link_w}" h="${base_link_h}" d="${base_link_d}"/>
-    <!-- <visual>
-      <origin
-        xyz="0 0 0"
-        rpy="0 0 0" />
-      <material name="black"/>
-    </visual> -->
-      <geometry>
-        <mesh
-          filename="file://$(find jetacker_description)/meshes/base_link.STL" />
-      </geometry>
-    <collision>
-      <surface>
-        <bounce>
-          <restitution_coefficient>0.0</restitution_coefficient>
-          <threshold>1.0</threshold>
-        </bounce>
-      </surface>
-      <origin
-        xyz="-0.004 0 ${base_link_d/2 + 0.022}"
-        rpy="0 0 0" />
-      <geometry>
-        <box size="${base_link_w} ${base_link_h} ${base_link_d}" />
-      </geometry>
-    </collision>
-  </link>
-  <link
-    name="back_shell_link">
-    <xacro:box_inertial m="${body_link_mass}" w="${body_link_w}" h="${body_link_h}" d="${body_link_d}"/>
-    <visual>
-      <origin
-        xyz="0 0 0"
-        rpy="0 0 0" />
-      <geometry>
-        <mesh
-          filename="file://$(find jetacker_description)/meshes/back_shell_link.STL" />
-      </geometry>
-      <material name="green"/>
-    </visual>
-    <collision>
-      <surface>
-        <bounce>
-          <restitution_coefficient>0.0</restitution_coefficient>
-          <threshold>1.0</threshold>
-        </bounce>
-      </surface>
-      <origin
-        xyz="-0.04 0 ${base_link_d + 0.022 + body_link_d/2}"
-        rpy="0 0 0" />
-      <geometry>
-        <box size="${body_link_w} ${body_link_h} ${body_link_d}" />
-      </geometry>
-    </collision>
-  </link>
-  <joint
-    name="back_shell_joint"
-    type="fixed">
-    <origin
-      xyz="0 0 0"
-      rpy="0 0 0" />
-    <parent
-      link="base_link" />
-    <child
-      link="back_shell_link" />
-    <axis
-      xyz="0 0 0" />
-  </joint>
-  <link
-    name="link1">
-    <inertial>
-      <origin
-        xyz="0.000273458158848059 4.49697391709507E-08 0.0127682239974202"
-        rpy="0 0 0" />
-      <mass
-        value="0.0117617552923888" />
-      <inertia
-        ixx="2.42304907313034E-06"
-        ixy="8.36427578709212E-13"
-        ixz="-4.88815706874446E-08"
-        iyy="2.24167366920736E-06"
-        iyz="2.4783598093895E-12"
-        izz="3.78066563706159E-06" />
-    </inertial>
-    <visual>
-      <origin
-        xyz="0 0 0"
-        rpy="0 0 0" />
-      <geometry>
-        <mesh
-          filename="file://$(find jetacker_description)/meshes/link1.STL" />
-      </geometry>
-      <material name="black"/>
-    </visual>
-  </link>
-  <joint
-    name="joint1"
-    type="revolute">
-    <origin
-      xyz="0.031299 0.00068637 0.16156"
-      rpy="0 0 0" />
-    <parent
-      link="base_link" />
-    <child
-      link="link1" />
-    <axis
-      xyz="0 0 1" />
-    <limit
-      lower="-2.09"
-      upper="2.09"
-      effort="1000"
-      velocity="10" />
-  </joint>
-  <link
-    name="depth_cam_link">
-    <inertial>
-      <origin
-        xyz="-0.00267477609208174 -1.63263137193841E-05 -0.00522210299748882"
-        rpy="0 0 0" />
-      <mass
-        value="0.22552781639362" />
-      <inertia
-        ixx="0.000408522155796754"
-        ixy="-7.65921501012663E-09"
-        ixz="1.66771046033071E-07"
-        iyy="4.81468336120099E-05"
-        iyz="-5.69880969191004E-09"
-        izz="0.000428962116485588" />
-    </inertial>
-    <visual>
-      <origin
-        xyz="0 0 0"
-        rpy="0 0 0" />
-      <geometry>
-        <mesh
-          filename="file://$(find jetacker_description)/meshes/depth_cam_link.STL" />
-      </geometry>
-      <material name="black"/>
-    </visual>
-  </link>
-  <joint
-    name="depth_cam_joint"
-    type="fixed">
-    <origin
-      xyz="0.0057651 0.00025 0.057913"
-      rpy="0 0 0" />
-    <parent
-      link="link1" />
-    <child
-      link="depth_cam_link" />
-    <axis
-      xyz="0 0 0" />
-  </joint>
-  <link
-    name="lidar_link">
-    <inertial>
-      <origin
-        xyz="-0.00221931680115031 0.000376419599582719 -0.0173018800523995"
-        rpy="0 0 0" />
-      <mass
-        value="0.0438457545362112" />
-      <inertia
-        ixx="1.59958556469832E-05"
-        ixy="4.53029353441676E-08"
-        ixz="2.33892337631863E-07"
-        iyy="2.04183700013467E-05"
-        iyz="-1.10000396493279E-08"
-        izz="3.50483610398295E-05" />
-    </inertial>
-    <visual>
-      <origin
-        xyz="0 0 0"
-        rpy="0 0 0" />
-      <geometry>
-        <mesh
-          filename="file://$(find jetacker_description)/meshes/lidar_link.STL" />
-      </geometry>
-      <material name="black"/>
-    </visual>
-  </link>
-  <joint
-    name="lidar_joint"
-    type="fixed">
-    <origin
-      xyz="0.10414 0.000685 0.13378"
-      rpy="0 0 0" />
-    <parent
-      link="base_link" />
-    <child
-      link="lidar_link" />
-    <axis
-      xyz="0 0 0" />
-  </joint>
-  <link name="lidar_sim_frame" />
-  <joint
-    name="lidar_sim_frame_joint"
-    type="fixed">
-    <origin xyz="0 0 0" rpy="0 0 ${M_PI}" />
-    <parent link="lidar_link" />
-    <child link="lidar_sim_frame" />
-  </joint>
-  <link
-    name="wheel_right_front">
-    <xacro:cylinder_inertial m="${wheel_link_mass}" r="${wheel_link_radius}" h="${wheel_link_length}" />
-    <visual>
-      <origin
-        xyz="0 0 0"
-        rpy="0 0 0" />
-      <geometry>
-        <mesh
-          filename="file://$(find jetacker_description)/meshes/wheel_right_front.STL" />
-      </geometry>
-      <material name="black"/>
-    </visual>
-    <collision>
-      <surface>
-        <bounce>
-          <restitution_coefficient>0.0</restitution_coefficient>
-          <threshold>1.0</threshold>
-        </bounce>
-      </surface>
-      <origin
-        xyz="0 -0.019 0"
-        rpy="${M_PI/2} 0 0" />
-      <geometry>
-        <cylinder length="${wheel_link_length}" radius="${wheel_link_radius}"/>
-      </geometry>
-    </collision>
-  </link>
-  <joint
-    name="wheel_right_front_joint"
-    type="fixed">
-    <origin
-      xyz="0.10733 -0.091241 0.050002"
-      rpy="0 0 0" />
-    <parent
-      link="base_link" />
-    <child
-      link="wheel_right_front" />
-    <axis
-      xyz="0 0 0" />
-  </joint>
-  <link
-    name="wheel_right_back">
-    <xacro:cylinder_inertial m="${wheel_link_mass}" r="${wheel_link_radius}" h="${wheel_link_length}" />
-    <visual>
-      <origin
-        xyz="0 0 0"
-        rpy="0 0 0" />
-      <geometry>
-        <mesh
-          filename="file://$(find jetacker_description)/meshes/wheel_right_back.STL" />
-      </geometry>
-      <material name="black"/>
-    </visual>
-    <collision>
-      <surface>
-        <bounce>
-          <restitution_coefficient>0.0</restitution_coefficient>
-          <threshold>1.0</threshold>
-        </bounce>
-      </surface>
-      <origin
-        xyz="0 -0.019 0"
-        rpy="${M_PI/2} 0 0" />
-      <geometry>
-        <cylinder length="${wheel_link_length}" radius="${wheel_link_radius}"/>
-      </geometry>
-    </collision>
-  </link>
-  <joint
-    name="wheel_right_back_joint"
-    type="fixed">
-    <origin
-      xyz="-0.106 -0.091444 0.050335"
-      rpy="0 0 0" />
-    <parent
-      link="base_link" />
-    <child
-      link="wheel_right_back" />
-    <axis
-      xyz="0 0 0" />
-  </joint>
-  <link
-    name="wheel_left_back">
-    <xacro:cylinder_inertial m="${wheel_link_mass}" r="${wheel_link_radius}" h="${wheel_link_length}" />
-    <visual>
-      <origin
-        xyz="0 0 0"
-        rpy="0 0 0" />
-      <geometry>
-        <mesh
-          filename="file://$(find jetacker_description)/meshes/wheel_left_back.STL" />
-      </geometry>
-      <material name="black"/>
-    </visual>
-    <collision>
-      <surface>
-        <bounce>
-          <restitution_coefficient>0.0</restitution_coefficient>
-          <threshold>1.0</threshold>
-        </bounce>
-      </surface>
-      <origin
-        xyz="0 0.019 0"
-        rpy="${M_PI/2} 0 0" />
-      <geometry>
-        <cylinder length="${wheel_link_length}" radius="${wheel_link_radius}"/>
-      </geometry>
-    </collision>
-  </link>
-  <joint
-    name="wheel_left_back_joint"
-    type="fixed">
-    <origin
-      xyz="-0.10599 0.090107 0.050328"
-      rpy="0 0 0" />
-    <parent
-      link="base_link" />
-    <child
-      link="wheel_left_back" />
-    <axis
-      xyz="0 0 0" />
-  </joint>
-  <link
-    name="wheel_left_front">
-    <xacro:cylinder_inertial m="${wheel_link_mass}" r="${wheel_link_radius}" h="${wheel_link_length}" />
-    <visual>
-      <origin
-        xyz="0 0 0"
-        rpy="0 0 0" />
-      <geometry>
-        <mesh
-          filename="file://$(find jetacker_description)/meshes/wheel_left_front.STL" />
-      </geometry>
-      <material name="black"/>
-    </visual>
-    <collision>
-      <surface>
-        <bounce>
-          <restitution_coefficient>0.0</restitution_coefficient>
-          <threshold>1.0</threshold>
-        </bounce>
-      </surface>
-      <origin
-        xyz="0 0.019 0"
-        rpy="${M_PI/2} 0 0" />
-      <geometry>
-        <cylinder length="${wheel_link_length}" radius="${wheel_link_radius}"/>
-      </geometry>
-    </collision>
-  </link>
-  <joint
-    name="wheel_left_front_joint"
-    type="fixed">
-    <origin
-      xyz="0.10734 0.092607 0.049998"
-      rpy="0 0 0" />
-    <parent
-      link="base_link" />
-    <child
-      link="wheel_left_front" />
-    <axis
-      xyz="0 0 0" />
-  </joint>
-</robot>
+/home/ubuntu/ros2_ws/build/jetacker_description/urdf/jetacker.urdf.xacro

File: install/jetacker_description/share/jetacker_description/urdf/jetacker.xacro (robot description, xacro)
@@ -1,14 +1 @@
-<?xml version="1.0" encoding="utf-8"?>
-<robot name="jetacker" xmlns:xacro="http://ros.org/wiki/xacro">
-    <xacro:property name="lidar"        value="$(env LIDAR_TYPE)"/>
-    <xacro:include filename="$(find jetacker_description)/urdf/materials.xacro"/>
-    <xacro:include filename="$(find jetacker_description)/urdf/inertial_matrix.xacro"/>
-    <xacro:include filename="$(find jetacker_description)/urdf/imu.urdf.xacro"/>
-    <xacro:if value="${lidar in ['A1', 'A2', 'S2L', 'LD14P']}">
-        <xacro:include filename="$(find jetacker_description)/urdf/lidar_a1.urdf.xacro"/>
-    </xacro:if>
-    <xacro:if value="${lidar in ['G4']}">
-        <xacro:include filename="$(find jetacker_description)/urdf/lidar_g4.urdf.xacro"/>
-    </xacro:if>
-    <xacro:include filename="$(find jetacker_description)/urdf/jetacker.urdf.xacro"/>
-</robot>
+/home/ubuntu/ros2_ws/build/jetacker_description/urdf/jetacker.xacro

File: install/jetacker_description/share/jetacker_description/urdf/lidar.gazebo.xacro (robot description, xacro)
@@ -1,35 +1 @@
-<?xml version="1.0" encoding="utf-8" ?>
-<robot name="lidar" xmlns:xacro="http://ros.org/wiki/xacro">
-    <xacro:property name="M_PI" value="3.1415926535897931"/>
-    <gazebo reference="lidar_frame">
-      <sensor type="ray" name="lidar">
-        <pose>0 0 0 0 0 0</pose>
-        <visualize>false</visualize>
-        <update_rate>5</update_rate>
-        <ray>
-          <scan>
-            <horizontal>
-              <samples>360</samples>
-              <resolution>1</resolution>
-              <min_angle>0</min_angle>
-              <max_angle>6.2832</max_angle>
-            </horizontal>
-          </scan>
-          <range>
-            <min>0.15</min>
-            <max>12</max>
-            <resolution>0.015</resolution>
-          </range>
-          <noise>
-            <type>gaussian</type>
-            <mean>0.0</mean>
-            <stddev>0.01</stddev>
-          </noise>
-        </ray>
-        <plugin name="gazebo_rplidar" filename="libgazebo_ros_laser.so">
-          <topicName>scan_raw</topicName>
-          <frameName>$(arg lidar_frame)</frameName>
-        </plugin>
-      </sensor>
-    </gazebo>
-</robot>
+/home/ubuntu/ros2_ws/build/jetacker_description/urdf/lidar.gazebo.xacro

File: install/jetacker_description/share/jetacker_description/urdf/lidar_a1.urdf.xacro (robot description, xacro)
@@ -1,12 +1 @@
-<?xml version="1.0" encoding="utf-8"?>
-<robot name="lidar_a1" xmlns:xacro="http://ros.org/wiki/xacro" >
-  <xacro:property name="M_PI" value="3.1415926535897931"/>
-  <link name="lidar_frame" />
-  <joint
-    name="lidar_frame_joint"
-    type="fixed">
-    <origin xyz="0 0 0" rpy="0 0 ${M_PI}" />
-    <parent link="lidar_link" />
-    <child link="lidar_frame" />
-  </joint>
-</robot>
+/home/ubuntu/ros2_ws/build/jetacker_description/urdf/lidar_a1.urdf.xacro

File: install/jetacker_description/share/jetacker_description/urdf/lidar_g4.urdf.xacro (robot description, xacro)
@@ -1,12 +1 @@
-<?xml version="1.0" encoding="utf-8"?>
-<robot name="lidar_g4" xmlns:xacro="http://ros.org/wiki/xacro" >
-  <xacro:property name="M_PI" value="3.1415926535897931"/>
-  <link name="lidar_frame" />
-  <joint
-    name="lidar_frame_joint"
-    type="fixed">
-    <origin xyz="0 0 0" rpy="0 0 0" />
-    <parent link="lidar_link" />
-    <child link="lidar_frame" />
-  </joint>
-</robot>
+/home/ubuntu/ros2_ws/build/jetacker_description/urdf/lidar_g4.urdf.xacro

File: install/jetacker_description/share/jetacker_description/urdf/materials.xacro (robot description, xacro)
@@ -1,27 +1 @@
-<?xml version="1.0"?>
-<robot name="material" xmlns:xacro="http://ros.org/wiki/xacro">
-    <material name="black">
-        <color rgba="0.1 0.1 0.1 1.0"/>
-    </material>
-    <material name="blue">
-        <color rgba="0.0 0.0 0.8 1.0"/>
-    </material>
-    <material name="green">
-        <color rgba="0.4 0.9 0.4 1.0"/>
-    </material>
-    <material name="gray">
-        <color rgba="0.7 0.7 0.7 1.0"/>
-    </material>
-    <material name="darkgray">
-        <color rgba="0.3 0.3 0.3 1.0"/>
-    </material>
-    <material name="red">
-        <color rgba="0.8 0.0 0.0 1.0"/>
-    </material>
-    <material name="white">
-        <color rgba="1.0 1.0 1.0 1.0"/>
-    </material>
-    <material name="yellow">
-        <color rgba="0.8 0.8 0.0 1.0"/>
-    </material>
-</robot>
+/home/ubuntu/ros2_ws/build/jetacker_description/urdf/materials.xacro

File: install/robot_gazebo/share/robot_gazebo/urdf/camera.gazebo.xacro (robot description, xacro)
@@ -1,24 +1 @@
-<?xml version="1.0" encoding="utf-8" ?>
-<robot name="camera_gazebo" xmlns:xacro="http://ros.org/wiki/xacro">
-  <gazebo reference="depth_cam_link">
-    <sensor name="robot_cam" type="camera">
-      <camera>
-        <horizontal_fov>1.047</horizontal_fov>
-        <image>
-          <width>640</width>
-          <height>400</height>
-        </image>
-        <clip>
-          <near>0.1</near>
-          <far>10</far>
-        </clip>
-      </camera>
-      <always_on>1</always_on>
-      <update_rate>30</update_rate>
-      <visualize>true</visualize>
-      <camera_info_topic>/depth_cam/rgb/camera_info</camera_info_topic>
-      <topic>/depth_cam/depth_cam</topic>
-      <enable_metrics>true</enable_metrics>
-    </sensor>
-  </gazebo>
-</robot>
+/home/ubuntu/ros2_ws/build/robot_gazebo/urdf/camera.gazebo.xacro

File: install/robot_gazebo/share/robot_gazebo/urdf/imu.gazebo.xacro (robot description, xacro)
@@ -1,12 +1 @@
-<?xml version="1.0" encoding="utf-8" ?>
-<robot xmlns:xacro="http://www.ros.org/wiki/xacro" name="robot_imu">
-    <gazebo reference="imu_link">
-        <sensor name="imu_sensor" type="imu">
-            <always_on>1</always_on>
-            <update_rate>50</update_rate>
-            <ignition_frame_id>imu_link</ignition_frame_id>
-            <visualize>true</visualize>
-            <topic>imu</topic>
-        </sensor>
-    </gazebo>
-</robot>
+/home/ubuntu/ros2_ws/build/robot_gazebo/urdf/imu.gazebo.xacro

File: install/robot_gazebo/share/robot_gazebo/urdf/jetacker.gazebo.xacro (robot description, xacro)
@@ -1,19 +1 @@
-<?xml version="1.0" encoding="utf-8"?>
-<robot name="car" xmlns:xacro="http://ros.org/wiki/xacro">
-  <ros2_control name="IgnitionSystem" type="system">
-    <hardware>
-      <plugin>ign_ros2_control/IgnitionSystem</plugin>
-    </hardware>
-    <joint name="joint1">
-      <command_interface name="position">
-        <param name="min">-2.09</param>
-        <param name="max">2.09</param>
-      </command_interface>
-      <state_interface name="position">
-        <param name="initial_value">0</param>
-      </state_interface>
-      <state_interface name="velocity"/>
-      <state_interface name="effort"/>
-    </joint>
-  </ros2_control>
-</robot>
+/home/ubuntu/ros2_ws/build/robot_gazebo/urdf/jetacker.gazebo.xacro

File: install/robot_gazebo/share/robot_gazebo/urdf/lidar.gazebo.xacro (robot description, xacro)
@@ -1,33 +1 @@
-<?xml version="1.0"?>
-<robot xmlns:xacro="http://www.ros.org/wiki/xacro" name="gpu_lidar">
-    <gazebo reference="lidar_link">
-        <sensor name="gpu_lidar" type="gpu_lidar">
-            <!--<pose relative_to='lidar_frame'>0 0 0 0 0 0</pose>-->
-            <topic>scan</topic>
-            <update_rate>10</update_rate>
-            <ignition_frame_id>lidar_link</ignition_frame_id>
-            <ray>
-                <scan>
-                    <horizontal>
-                        <samples>360</samples>
-                        <resolution>1</resolution>
-                        <min_angle>-3.14159</min_angle>
-                        <max_angle>3.14159</max_angle>
-                    </horizontal>
-                </scan>
-                <range>
-                    <min>0.10</min>
-                    <max>12.0</max>
-                    <resolution>0.01</resolution>
-                </range>
-                <noise>
-                    <type>gaussian</type>
-                    <mean>0.0</mean>
-                    <stddev>0.01</stddev>
-                </noise>
-            </ray>
-            <alwaysOn>1</alwaysOn>
-            <visualize>true</visualize>
-        </sensor>
-    </gazebo>
-</robot>
+/home/ubuntu/ros2_ws/build/robot_gazebo/urdf/lidar.gazebo.xacro
