Commit message: 08/08/2025

File: install/robot_gazebo/share/robot_gazebo/urdf/robot.gazebo.xacro (robot description, xacro)
@@ -1,50 +1 @@
-<?xml version="1.0" encoding="utf-8"?>
-<robot name="robot" xmlns:xacro="http://ros.org/wiki/xacro">
-    <xacro:arg name="sim_ign" default="true"/>
-    <!-- robot_description -->
-    <xacro:include filename="$(find jetacker_description)/urdf/jetacker.xacro"/>
-    <xacro:if value="$(arg sim_ign)">
-        <xacro:include filename="$(find robot_gazebo)/urdf/wheel_base.urdf.xacro"/>
-    </xacro:if>
-    <!-- ign_joint_control -->
-    <xacro:include filename="$(find robot_gazebo)/urdf/jetacker.gazebo.xacro"/>
-    <!-- lidar -->
-    <xacro:include filename="$(find robot_gazebo)/urdf/lidar.gazebo.xacro"/>
-    <!-- camera -->
-    <xacro:include filename="$(find robot_gazebo)/urdf/camera.gazebo.xacro"/>
-    <gazebo>
-        <!-- Joint state publisher -->
-        <plugin filename="$(find ign_ros2_control)/../../lib/libign_ros2_control-system.so"
-                name="ign_ros2_control::IgnitionROS2ControlPlugin">
-          <parameters>$(find robot_gazebo)/config/robot_config.yaml</parameters>
-        </plugin>
-        <!-- joint -->
-        <plugin filename="libignition-gazebo-joint-state-publisher-system.so" name="ignition::gazebo::systems::JointStatePublisher">
-            <topic>joint_states</topic>
-        </plugin>
-        <!-- sensor-lidar -->
-        <plugin filename="ignition-gazebo-sensors-system" name="ignition::gazebo::systems::Sensors">
-            <render_engine>ogre2</render_engine>
-        </plugin>
-        <!-- imu -->
-        <plugin filename="ignition-gazebo-imu-system" name="ignition::gazebo::systems::Imu"></plugin>
-        <!-- odom -->
-        <plugin
-            filename="ignition-gazebo-odometry-publisher-system"
-            name="ignition::gazebo::systems::OdometryPublisher">
-            <odom_publish_frequency>50</odom_publish_frequency>
-            <odom_topic>/odom</odom_topic>
-            <odom_frame>odom</odom_frame>
-            <robot_base_frame>base_footprint</robot_base_frame>
-            <tf_topic>/odom/tf</tf_topic>
-        </plugin>
-        <!-- Holonomic plugin -->
-        <xacro:if value="$(arg sim_ign)">
-            <plugin filename="libHolonomicPlugin.so" name="holonomic_sim::HolonomicPlugin">
-                <wheel_joint>wheel_joint</wheel_joint>
-                <top_base_joint>top_wheel_base_joint</top_base_joint>
-                <bottom_base_joint>bottom_wheel_base_joint</bottom_base_joint>
-            </plugin>
-        </xacro:if>
-    </gazebo>
-</robot>
+/home/ubuntu/ros2_ws/build/robot_gazebo/urdf/robot.gazebo.xacro

File: install/robot_gazebo/share/robot_gazebo/urdf/wheel_base.urdf.xacro (robot description, xacro)
@@ -1,57 +1 @@
-<?xml version="1.0" encoding="utf-8"?>
-<robot name="wheel_base" xmlns:xacro="http://ros.org/wiki/xacro" >
-    <xacro:macro name="cylinder_link_macro" params="suffix mass arg radius length if_collision if_visual">
-        <xacro:property name="sq_r" value="${radius*radius}"/>
-        <xacro:property name="sq_l" value="${length*length}"/>
-        <link name="${suffix}_link">
-            <inertial>
-                <mass value="${mass}"/>
-                <origin xyz="0 0 0" rpy="0 0 0"/>
-                <inertia ixx="${3*sq_r*arg/12+sq_l*arg/12}" ixy="0.0" ixz="0.0" iyy="${3*sq_r*arg/12+sq_l*arg/12}"
-                iyz="0.0" izz="${arg*sq_r/2}"/>
-            </inertial>
-            <xacro:if value="${if_visual}">
-                <visual>
-                    <geometry>
-                        <cylinder length="${length}" radius="${radius}"/>
-                    </geometry>
-                    <material name="red">
-                        <color rgba="1.0 0.0 0.0 1.0"/>
-                    </material>
-                </visual>
-            </xacro:if>
-            <xacro:if value="${if_collision}">
-                <collision>
-                    <geometry>
-                        <cylinder length="${length}" radius="${radius}"/>
-                    </geometry>
-                    <origin xyz="0 0 0" rpy="0 0 0"/>
-                </collision>
-            </xacro:if>
-        </link>
-    </xacro:macro>
-    <xacro:macro name="steer_macro" params="suffix parent base_radius wheel_radius wheel_offset x y z">
-        <xacro:cylinder_link_macro suffix="top_${suffix}_base" mass="0.0001" arg="1.0" radius="${base_radius}" length="0.001" if_collision="false" if_visual="false"/>
-        <joint name="top_${suffix}_base_joint" type="continuous">
-            <parent link="${parent}"/>
-            <child  link="top_${suffix}_base_link"/>
-            <origin xyz="${x} ${y} ${z+0.1}" rpy="0 0 0"/>
-            <axis xyz="0 0 1"/>
-        </joint>
-        <xacro:cylinder_link_macro suffix="bottom_${suffix}_base" mass="0.0001" arg="100000.0" radius="${base_radius}" length="0.001" if_collision="false" if_visual="false"/>
-        <joint name="bottom_${suffix}_base_joint" type="continuous">
-            <parent link="top_${suffix}_base_link"/>
-            <child  link="bottom_${suffix}_base_link"/>
-            <origin xyz="${x} ${y} ${z-0.1}" rpy="0 0 0"/>
-            <axis xyz="0 0 1"/>
-        </joint>
-        <xacro:cylinder_link_macro suffix="${suffix}" mass="0.0001" arg="0.0001" radius="${wheel_radius}" length="0.001" if_collision="true" if_visual="false"/>
-        <joint name="${suffix}_joint" type="continuous">
-            <parent link="bottom_${suffix}_base_link"/>
-            <child  link="${suffix}_link"/>
-            <origin xyz="0 0 ${wheel_offset}" rpy="-1.57 0 0"/>
-            <axis xyz="0 0 1"/>
-        </joint>
-    </xacro:macro>
-    <xacro:steer_macro suffix="wheel" parent="base_footprint" base_radius="0.3" wheel_radius="0.178" x="0" y="0" z="0" wheel_offset="0.1735"/>
-</robot>
+/home/ubuntu/ros2_ws/build/robot_gazebo/urdf/wheel_base.urdf.xacro
